File: light-meter-A.sch (EAGLE design)
At the start: 53 parts, among them IC1 ATMEGA328P, IC2 MCP73831, IC4 MCP1700-33, J1 AYZ0202, J2 AYZ0202, Q4 BSS123, Q5 BSS123, Q6 BSS123, Q7 BSS123, U1 MLX90614_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

Commit message: tighter board
Parts:
- removed LED4, LED5: RGBLED5050, adafruit:RGBLED5050
- removed RN6, RN7: (no value), resistor-dil:4R-NEXB38V
Connections:
- removed net N$21: LED4.BLUE_A, RN6C.1
- removed net N$22: LED4.GREEN_A, RN6B.1
- removed net N$23: LED4.RED_A, RN6A.1
- removed net N$24: LED5.BLUE_A, RN7C.1
- removed net N$25: LED5.GREEN_A, RN7B.1
- removed net N$26: LED5.RED_A, RN7A.1
- net BLUE: no longer RN6B.2, RN7B.2
- net GND: now also N1.8; no longer LED4.BLUE_C, LED4.GREEN_C, LED4.RED_C, LED5.BLUE_C, LED5.GREEN_C, LED5.RED_C
- net GREEN: no longer RN6C.2, RN7C.2
- net RED: no longer RN6A.2, RN7A.2
Changed lines of the file:
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@@
 <part name="GND10" library="supply1" deviceset="GND" device=""/>
 <part name="RN5" library="resistor-dil" deviceset="4R-N" device="EXB38V"/>
-<part name="LED4" library="adafruit" deviceset="RGBLED" device="5050"/>
-<part name="GND11" library="supply1" deviceset="GND" device=""/>
-<part name="RN6" library="resistor-dil" deviceset="4R-N" device="EXB38V"/>
-<part name="LED5" library="adafruit" deviceset="RGBLED" device="5050"/>
-<part name="GND12" library="supply1" deviceset="GND" device=""/>
-<part name="RN7" library="resistor-dil" deviceset="4R-N" device="EXB38V"/>
 <part name="SUPPLY1" library="supply2" deviceset="GND" device=""/>
 <part name="P+8" library="supply1" deviceset="VCC" device=""/>
@@
 <instance part="RN5" gate="B" x="195.834" y="-49.276"/>
 <instance part="RN5" gate="C" x="196.088" y="-54.356"/>
-<instance part="LED4" gate="G$1" x="125.476" y="-82.042" rot="R180"/>
-<instance part="GND11" gate="1" x="120.396" y="-96.52"/>
-<instance part="RN6" gate="A" x="140.208" y="-76.962"/>
-<instance part="RN6" gate="B" x="140.208" y="-82.042"/>
-<instance part="RN6" gate="C" x="140.462" y="-87.122"/>
-<instance part="LED5" gate="G$1" x="180.086" y="-81.788" rot="R180"/>
-<instance part="GND12" gate="1" x="175.006" y="-96.266"/>
-<instance part="RN7" gate="A" x="194.818" y="-76.708"/>
-<instance part="RN7" gate="B" x="194.818" y="-81.788"/>
-<instance part="RN7" gate="C" x="195.072" y="-86.868"/>
 <instance part="SUPPLY1" gate="GND" x="262.636" y="-10.922"/>
 <instance part="P+8" gate="VCC" x="262.636" y="12.954"/>
@@
 </segment>
 <segment>
-<wire x1="423.672" y1="143.51" x2="430.022" y2="143.51" width="0.1524" layer="91"/>
+<wire x1="423.672" y1="143.51" x2="423.926" y2="143.51" width="0.1524" layer="91"/>
 <label x="429.006" y="144.018" size="1.778" layer="95"/>
+<pinref part="N1" gate="1" pin="8"/>
+<wire x1="423.926" y1="143.51" x2="430.022" y2="143.51" width="0.1524" layer="91"/>
 </segment>
 <segment>
@@
 <junction x="176.022" y="-54.356"/>
 <pinref part="GND10" gate="1" pin="GND"/>
-</segment>
-<segment>
-<pinref part="LED4" gate="G$1" pin="RED_C"/>
-<pinref part="LED4" gate="G$1" pin="GREEN_C"/>
-<pinref part="LED4" gate="G$1" pin="BLUE_C"/>
-<wire x1="120.396" y1="-87.122" x2="120.396" y2="-82.042" width="0.1524" layer="91"/>
-<junction x="120.396" y="-82.042"/>
-<wire x1="120.396" y1="-82.042" x2="120.396" y2="-76.962" width="0.1524" layer="91"/>
-<wire x1="120.396" y1="-87.122" x2="120.396" y2="-93.98" width="0.1524" layer="91"/>
-<junction x="120.396" y="-87.122"/>
-<pinref part="GND11" gate="1" pin="GND"/>
-</segment>
-<segment>
-<pinref part="LED5" gate="G$1" pin="RED_C"/>
-<pinref part="LED5" gate="G$1" pin="GREEN_C"/>
-<pinref part="LED5" gate="G$1" pin="BLUE_C"/>
-<wire x1="175.006" y1="-86.868" x2="175.006" y2="-81.788" width="0.1524" layer="91"/>
-<junction x="175.006" y="-81.788"/>
-<wire x1="175.006" y1="-81.788" x2="175.006" y2="-76.708" width="0.1524" layer="91"/>
-<wire x1="175.006" y1="-86.868" x2="175.006" y2="-93.726" width="0.1524" layer="91"/>
-<junction x="175.006" y="-86.868"/>
-<pinref part="GND12" gate="1" pin="GND"/>
 </segment>
 <segment>
@@
 <label x="205.74" y="-44.196" size="1.778" layer="95"/>
 </segment>
-<segment>
-<pinref part="RN6" gate="A" pin="2"/>
-<wire x1="145.288" y1="-76.962" x2="149.86" y2="-76.962" width="0.1524" layer="91"/>
-<label x="150.114" y="-76.962" size="1.778" layer="95"/>
-</segment>
-<segment>
-<pinref part="RN7" gate="A" pin="2"/>
-<wire x1="199.898" y1="-76.708" x2="204.47" y2="-76.708" width="0.1524" layer="91"/>
-<label x="204.724" y="-76.708" size="1.778" layer="95"/>
-</segment>
 </net>
 <net name="GREEN" class="0">
@@
 <label x="206.248" y="-54.102" size="1.778" layer="95"/>
 </segment>
-<segment>
-<pinref part="RN6" gate="C" pin="2"/>
-<wire x1="145.542" y1="-87.122" x2="150.114" y2="-87.122" width="0.1524" layer="91"/>
-<label x="150.622" y="-86.868" size="1.778" layer="95"/>
-</segment>
-<segment>
-<pinref part="RN7" gate="C" pin="2"/>
-<wire x1="200.152" y1="-86.868" x2="204.724" y2="-86.868" width="0.1524" layer="91"/>
-<label x="205.232" y="-86.614" size="1.778" layer="95"/>
-</segment>
 </net>
 <net name="BLUE" class="0">
@@
 <wire x1="200.914" y1="-49.276" x2="205.486" y2="-49.276" width="0.1524" layer="91"/>
 <label x="205.486" y="-49.022" size="1.778" layer="95"/>
-</segment>
-<segment>
-<pinref part="RN6" gate="B" pin="2"/>
-<wire x1="145.288" y1="-82.042" x2="149.86" y2="-82.042" width="0.1524" layer="91"/>
-<label x="149.86" y="-81.788" size="1.778" layer="95"/>
-</segment>
-<segment>
-<pinref part="RN7" gate="B" pin="2"/>
-<wire x1="199.898" y1="-81.788" x2="204.47" y2="-81.788" width="0.1524" layer="91"/>
-<label x="204.47" y="-81.534" size="1.778" layer="95"/>
 </segment>
 </net>
@@
 </segment>
 </net>
-<net name="N$21" class="0">
-<segment>
-<pinref part="LED4" gate="G$1" pin="BLUE_A"/>
-<pinref part="RN6" gate="C" pin="1"/>
-<wire x1="135.382" y1="-87.122" x2="130.556" y2="-87.122" width="0.1524" layer="91"/>
-</segment>
-</net>
-<net name="N$22" class="0">
-<segment>
-<pinref part="LED4" gate="G$1" pin="GREEN_A"/>
-<pinref part="RN6" gate="B" pin="1"/>
-<wire x1="135.128" y1="-82.042" x2="130.556" y2="-82.042" width="0.1524" layer="91"/>
-</segment>
-</net>
-<net name="N$23" class="0">
-<segment>
-<pinref part="LED4" gate="G$1" pin="RED_A"/>
-<pinref part="RN6" gate="A" pin="1"/>
-<wire x1="135.128" y1="-76.962" x2="130.556" y2="-76.962" width="0.1524" layer="91"/>
-</segment>
-</net>
-<net name="N$24" class="0">
-<segment>
-<pinref part="LED5" gate="G$1" pin="BLUE_A"/>
-<pinref part="RN7" gate="C" pin="1"/>
-<wire x1="189.992" y1="-86.868" x2="185.166" y2="-86.868" width="0.1524" layer="91"/>
-</segment>
-</net>
-<net name="N$25" class="0">
-<segment>
-<pinref part="LED5" gate="G$1" pin="GREEN_A"/>
-<pinref part="RN7" gate="B" pin="1"/>
-<wire x1="189.738" y1="-81.788" x2="185.166" y2="-81.788" width="0.1524" layer="91"/>
-</segment>
-</net>
-<net name="N$26" class="0">
-<segment>
-<pinref part="LED5" gate="G$1" pin="RED_A"/>
-<pinref part="RN7" gate="A" pin="1"/>
-<wire x1="189.738" y1="-76.708" x2="185.166" y2="-76.708" width="0.1524" layer="91"/>
-</segment>
-</net>
