File: open-lab-VUSB-A.sch (EAGLE design)
At the start: 49 parts, among them IC1 ATMEGA328P, IC2 MCP73831, IC4 MCP1700-33, J1 AYZ0202, Q4 BSS123, Q5 BSS123, Q6 BSS123, Q7 BSS123, U1 MLX90614_, X1 USBSMD

Commit message: update
Parts:
- removed BAT1: LIR2032, SparkFunNew:BATTERYBATTCOM_20MM_PTH_SMT
- removed BTN: EVQQ2, adafruit:EVQQ2
- removed C14, C15: 0.1uF, adafruit:C-USC0805
- removed J2: (no value), jumper:JP1E
- removed LED, LED1, LED2, LED3: RGBLED5050, adafruit:RGBLED5050
- removed LUXNIR: TSL2561, microbuilder:TSL2561
- removed LUXRGB: TCS34725, dwbLibrary:TCS34725
- removed N1, SV2: (no value), con-lstb:MA08-1
- removed Q4, Q5, Q6, Q7: BSS123, transistor-small-signal:BSS123
- removed R14, R15: 10K, adafruit:R-US_R0805
- removed RIR1, RIR2: 10K, rcl:R-EU_R0805
- removed RN2, RN4, RN5: (no value), resistor-dil:4R-NEXB38V
- removed U$1: BUZZER, adafruit:BUZZER
- removed U1: MLX90614_, SparkFun:MLX90614_
- added C11: 0.1u, rcl:C-EUC0805
- added C12, C13: 0.1µ, resistor:C-EUC0805
- added CAP: 10u, resistor:C-EUC0805
- added CPR: 1.0uF, adafruit:C-USC0805
- added CTC1, CTC2: 10uF, adafruit:C-USC0805K
- added CTCP: 0.01µF, microbuilder:CAP_CERAMIC_0805
- added CX3, CX4: 18p, resistor:C-EUC0805
- added D1: 1N4148, adafruit:DIODESOD-323F
- added D2: 1n4148, adafruit:DIODESOD-323F
- added DHT22: (no value), SparkFun-Connectors:M04LOCK
- added ETH, LCD: (no value), jumper:JP1E
- added FB1, FB2: Ferrite, microbuilder:FERRITE_0805
- added IC6: MAX31855, adafruit:MAX6675
- added IC7: ENC28J60, SparkFun:ENC28J60SO28LONG
- added L1: Bead, rcl:R-EU_R0805
- added MICROSD: USD-SOCKETMICRO-SD-SOCKET-TAOBAO, SparkFunNew:USD-SOCKETMICRO-SD-SOCKET-TAOBAO
- added N5110: (no value), con-lstb:MA08-1
- added Q2: BSS123, transistor-small-signal:BSS123
- added RBS: 2.32K, rcl:R-EU_R0805
- added REA1, REB1: 330, rcl:R-EU_R0805
- added RH: 10k, rcl:R-US_R0805
- added RJ45: HR911105A, CONNECTER:HR911105A
- added RM3, RM4: 1.5K, rcl:R-EU_R0805
- added RR+, RR-, RT+, RT-: 49.9, rcl:R-EU_R0805
- added RSD: 10K, rcl:R-EU_R0805
- added RTC: DS1307, adafruit:DS1307SOIC
- added RTCP1, RTCP2: 10K, adafruit:R-US_R0805
- added RTHM2: 3k, rcl:R-US_R0805
- added TCPL, THM2: 1X2-3.5MM, adafruit:1X2-3.5MM
- added U3: BMP085, microbuilder:BMP085
- added UART: (no value), con-lstb:MA04-1
- added X2: 32.768kHz, crystal:CRYSTALTC26H
- added X3: 25MHz, SparkFun:CRYSTALHC49UV
Connections:
- removed net +3V3: C14.1, C15.1, LUXNIR.3.3V, LUXRGB.VDD, R14.2, R15.2
- removed net A4: IC1.PC4(ADC4/SDA)
- removed net A5: IC1.PC5(ADC5/SCL)
- removed net BLUE: Q6.S, RN2B.2, RN3B.2, RN4B.2, RN5B.2
- removed net GREEN: Q7.S, RN2C.2, RN3C.2, RN4C.2, RN5C.2
- removed net N$13: LED1.GREEN_A, RN3B.1
- removed net N$14: LED1.RED_A, RN3A.1
- removed net N$15: LED2.BLUE_A, RN4C.1
- removed net N$16: LED2.GREEN_A, RN4B.1
- removed net N$17: LED2.RED_A, RN4A.1
- removed net N$18: LED3.BLUE_A, RN5C.1
- removed net N$19: LED3.GREEN_A, RN5B.1
- removed net N$20: LED3.RED_A, RN5A.1
- removed net N$4: LED.BLUE_A, RN2C.1
- removed net N$7: Q4.D, U$1.-
- removed net RED: Q5.S, RN2A.2, RN3A.2, RN4A.2, RN5A.2
- removed net RGB-INT: LUXRGB.INT
- removed net VIS-NIR-ADDR: LUXNIR.ADDRSEL
- removed net VIS-NIR-INT: LUXNIR.INT
- new net CS: D1.A, IC6./CS, RTCP2.2
- new net LEDA: REA1.2, RJ45.G+
- new net LEDB: REB1.2, RJ45.Y+
- new net N$21: RTC.X1, X2.2
- new net N$30: RTC.X2, X2.1
- new net N$34: IC7.LEDA, REA1.1
- new net N$37: IC7.LEDB, REB1.1
- new net N$39: CAP.1, IC7.VCAP
- new net N$41: CX3.1, IC7.OSC2, X3.2
- new net N$42: CX4.1, IC7.OSC1, X3.1
- new net N$54: C13.2, RR+.2, RR-.1
- new net N$59: IC7.RBIAS, RBS.2
- new net RD+: IC7.TPIN+, RJ45.RD+, RR+.1
- new net RD-: IC7.TPIN-, RJ45.RD-, RR-.2
- new net SCK1: D2.A, IC6.SCK, RTCP1.2
- new net TCT: C12.2, L1.1, RJ45.P4, RT+.2, RT-.1
- new net TD+: IC7.TPOUT+, RJ45.TD+, RT+.1
- new net TD-: IC7.TPOUT-, RJ45.TD-, RT-.2
- new net V_CON: ETH.2, IC7.VDD, IC7.VDDOSC, IC7.VDDPLL, IC7.VDDRX, IC7.VDDTX, LCD.2, N5110.6, N5110.7, Q2.D, RM4.2
- net A0: now also RTHM1.2, THM1.1; no longer SV2.7
- net A1: now also RTHM2.2, THM2.1; no longer SV2.8
- net A2: now also RM3.2, RM4.1; no longer RTHM1.2, THM1.1
- net A3: now also MICROSD.CS, RSD.1; no longer BTN.S, BTN.S1
- net D10: no longer Q7.G
- net D2: now also N5110.3
- net D3: now also N5110.4; no longer N1.3
- net D4: now also N5110.5; no longer N1.4
- net D5: no longer N1.5
- net D6: now also D1.C; no longer Q5.G
- net D8: now also IC7.CS; no longer Q6.G
- net D9: now also DHT22.2, RH.2; no longer Q4.G
- net GND: now also C11.2, C12.1, C13.1, CAP.2, CPR.2, CTC1.2, CTC2.2, CX3.2, CX4.2, DHT22.4, IC6.GND, IC7.VSS, IC7.VSSOSC, IC7.VSSPLL, IC7.VSSRX, IC7.VSSTX, MICROSD.GND, MICROSD.SHIELD@1, MICROSD.SHIELD@2, MICROSD.SHIELD@3, MICROSD.SHIELD@4, N5110.2, RBS.1, RJ45.G-, RJ45.GND, RJ45.SHIELD0, RJ45.SHIELD1, RJ45.Y-, RM3.1, RTC.GND, RTHM2.1, U3.GND, UART.1; no longer BAT1.-, BTN.P, BTN.P1, C14.2, C15.2, LED.BLUE_C, LED.GREEN_C, LED.RED_C, LED1.BLUE_C, LED1.GREEN_C, LED1.RED_C, LED2.BLUE_C, LED2.GREEN_C, LED2.RED_C, LED3.BLUE_C, LED3.GREEN_C, LED3.RED_C, LUXNIR.GND, LUXRGB.GND, N1.2, N1.8, Q4.S, SV2.1, U1.VSS
- net MISO: now also IC6.DO, IC7.SO, MICROSD.DO
- net MOSI: now also IC7.SI, MICROSD.DI
- net N$11: now also FB2.P$1, TCPL.1; no longer LED.RED_A, RN2A.1
- net N$12: now also CTCP.P$2, FB2.P$2, IC6.T+; no longer LED1.BLUE_A, RN3C.1
- net N$8: now also FB1.P$1, TCPL.2; no longer J2.2, N1.7
- net N$9: now also CTCP.P$1, FB1.P$2, IC6.T-; no longer LED.GREEN_A, RN2B.1
- net RESET: now also IC7.RESET, N5110.1; no longer N1.1
- net RXD: now also UART.3; no longer SV2.3
- net SCK: now also D2.C, IC7.SCK, MICROSD.SCK
- net SCL: now also IC1.PC5(ADC5/SCL), RN3A.1, RTC.SCL, U3.SCL; no longer LUXNIR.SCL, LUXRGB.SCL, R15.1, RIR2.1, SV2.6, U1.SCL/VZ
- net SDA: now also IC1.PC4(ADC4/SDA), RN3B.1, RTC.SDA, U3.SDA; no longer LUXNIR.SDA, LUXRGB.SDA, R14.1, RIR1.1, SV2.5, U1.PWM/SDA
- net TXD: now also UART.4; no longer SV2.4
- net VBAT: no longer BAT1.+
- net VBUS: now also Q2.G
- net VCC: now also C11.1, CPR.1, CTC1.1, CTC2.1, DHT22.1, ETH.1, IC6.VCC, L1.2, LCD.1, MICROSD.VCC, Q2.S, RH.1, RN3A.2, RN3B.2, RSD.2, RTC.VBAT, RTC.VCC, RTCP1.1, RTCP2.1, THM2.2, U3.AVDD, U3.VDD, UART.2; no longer J2.1, N1.6, Q5.D, Q6.D, Q7.D, RIR1.2, RIR2.2, SV2.2, U$1.+, U1.VDD
Other:
- note added: "DHT22 - Temp and Humidity"
- note added: "Pressure"
- note added: "RTC"
- note removed: "RGB+Clear"
- note removed: "White + NIR"
- moved on the sheet: RN3A, RN3B, RTHM1
