File: open-lab-mon-A-mini.sch (EAGLE design)
At the start: 49 parts, among them IC1 ATMEGA328P, IC2 MCP73831, IC4 MCP1700-33, J1 AYZ0202, Q4 BSS123, Q5 BSS123, Q6 BSS123, Q7 BSS123, U1 MLX90614_, X1 USBSMD

Commit message: update
Parts:
- removed C15: 0.1uF, adafruit:C-USC0805
- removed LED, LED1, LED2, LED3: RGBLED5050, adafruit:RGBLED5050
- removed LUXNIR: TSL2561, microbuilder:TSL2561
- removed LUXRGB: TCS34725, dwbLibrary:TCS34725
- removed N1, SV2: (no value), con-lstb:MA08-1
- removed Q5, Q6, Q7: BSS123, transistor-small-signal:BSS123
- removed R14, R15: 10K, adafruit:R-US_R0805
- removed RIR1, RIR2: 10K, rcl:R-EU_R0805
- removed RN3, RN4, RN5: (no value), resistor-dil:4R-NEXB38V
- removed RTHM1: 3k, rcl:R-US_R0805
- removed THM1: 1X2-3.5MM, adafruit:1X2-3.5MM
- removed U1: MLX90614_, SparkFun:MLX90614_
- added C10, C9: 0.1µ, resistor:C-EUC0805
- added C6, C7: 10uF, adafruit:C-USC0805K
- added C8: 0.01µF, microbuilder:CAP_CERAMIC_0805
- added CAP1: 10u, resistor:C-EUC0805
- added CX1, CX2: 18p, resistor:C-EUC0805
- added D1: 1N4148, adafruit:DIODESOD-323F
- added D2: 1n4148, adafruit:DIODESOD-323F
- added FB1, FB2: Ferrite, microbuilder:FERRITE_0805
- added IC3: ENC28J60, SparkFun:ENC28J60SO28LONG
- added IC6: MAX31855, adafruit:MAX6675
- added J3, J4, J5: 1X2-3.5MM, adafruit:1X2-3.5MM
- added JP3: (no value), SparkFun-Connectors:M04LOCK
- added L2: Bead, rcl:R-EU_R0805
- added N5110: (no value), con-lstb:MA08-1
- added R1, R10, R6, R7: 3K, adafruit:R-US_R0805
- added R11, R3: 47K, adafruit:R-US_R0805
- added R2: 10K, rcl:R-EU_R0805
- added R4, R5: 10K, adafruit:R-US_R0805
- added RBS1: 2.32K, rcl:R-EU_R0805
- added REA, REB: 330, rcl:R-EU_R0805
- added RJ1: HR911105A, CONNECTER:HR911105A
- added RL: PHOTOCELL, SparkFunNew:PHOTOCELLPTH
- added U3: BMP085, microbuilder:BMP085
- added X2A: 25MHz, SparkFun:CRYSTAL10.5X4.8
- C14: value 0.1uF -> 1.0uF
- J2: value (none) -> 1X2-3.5MM; device jumper:JP1E -> adafruit:1X2-3.5MM
- RN2: value (none) -> 49.9
Connections:
- removed net A4: IC1.PC4(ADC4/SDA)
- removed net A5: IC1.PC5(ADC5/SCL)
- removed net BLUE: Q6.S, RN2B.2, RN3B.2, RN4B.2, RN5B.2
- removed net GREEN: Q7.S, RN2C.2, RN3C.2, RN4C.2, RN5C.2
- removed net RED: Q5.S, RN2A.2, RN3A.2, RN4A.2, RN5A.2
- removed net RGB-INT: LUXRGB.INT
- removed net VIS-NIR-ADDR: LUXNIR.ADDRSEL
- removed net VIS-NIR-INT: LUXNIR.INT
- new net 3.3V: JP3.1, R10.2
- new net AIO: J3.2, J4.2, J5.2, R1.1, R6.1, R7.1
- new net CS: D1.A, IC6./CS, R5.2
- new net DIO: JP3.2, R10.1
- new net DIO-0: D2.C
- new net E-CLK: IC3.CLKOUT
- new net E-INT: IC3./INT
- new net LEDA: REA.2, RJ1.G+
- new net LEDB: REB.2, RJ1.Y+
- new net N$22: N5110.5
- new net N$23: N5110.4
- new net N$24: N5110.3
- new net N$25: N5110.2
- new net N$26: N5110.1
- new net RD+: IC3.TPIN+, RJ1.RD+, RN2D.1
- new net RD-: IC3.TPIN-, RJ1.RD-, RN2C.1
- new net SCK1: D2.A, IC6.SCK, R4.2
- new net SCL1: R3.2
- new net SDA1: R11.2
- new net TCT: C10.2, L2.1, RJ1.P4, RN2A.2, RN2B.2
- new net TD+: IC3.TPOUT+, RJ1.TD+, RN2B.1
- new net TD-: IC3.TPOUT-, RJ1.TD-, RN2A.1
- net +3V3: now also C6.1, C7.1, IC3.VDD, IC3.VDDOSC, IC3.VDDPLL, IC3.VDDRX, IC3.VDDTX, IC6.VCC, J3.1, J4.1, J5.1, R4.1, R5.1, U3.AVDD, U3.VDD; no longer C15.1, LUXNIR.3.3V, LUXRGB.VDD, R14.2, R15.2
- net A0: now also R2.1, RL.P$1; no longer SV2.7
- net A1: no longer SV2.8
- net A2: no longer RTHM1.2, THM1.1
- net A3: no longer BTN.S, BTN.S1
- net D10: no longer Q7.G
- net D3: no longer N1.3
- net D4: now also BTN.S, BTN.S1; no longer N1.4
- net D5: no longer N1.5
- net D6: no longer Q5.G
- net D8: now also IC3.CS; no longer Q6.G
- net GND: now also C10.1, C6.2, C7.2, C9.1, CAP1.2, CX1.2, CX2.2, IC3.VSS, IC3.VSSOSC, IC3.VSSPLL, IC3.VSSRX, IC3.VSSTX, IC6.GND, JP3.4, R1.2, R2.2, R6.2, R7.2, RBS1.1, RJ1.G-, RJ1.GND, RJ1.SHIELD0, RJ1.SHIELD1, RJ1.Y-, U3.GND; no longer C15.2, LED.BLUE_C, LED.GREEN_C, LED.RED_C, LED1.BLUE_C, LED1.GREEN_C, LED1.RED_C, LED2.BLUE_C, LED2.GREEN_C, LED2.RED_C, LED3.BLUE_C, LED3.GREEN_C, LED3.RED_C, LUXNIR.GND, LUXRGB.GND, N1.2, N1.8, RTHM1.1, SV2.1, U1.VSS
- net MISO: now also IC3.SO, IC6.DO
- net MOSI: now also IC3.SI
- net N$11: now also FB2.P$1, J2.1; no longer LED.RED_A, RN2A.1
- net N$12: now also C8.P$2, FB2.P$2, IC6.T+; no longer LED1.BLUE_A, RN3C.1
- net N$13: now also N5110.8; no longer LED1.GREEN_A, RN3B.1
- net N$14: now also IC3.LEDA, REA.1; no longer LED1.RED_A, RN3A.1
- net N$15: now also IC3.LEDB, REB.1; no longer LED2.BLUE_A, RN4C.1
- net N$16: now also CAP1.1, IC3.VCAP; no longer LED2.GREEN_A, RN4B.1
- net N$17: now also IC3.RBIAS, RBS1.2; no longer LED2.RED_A, RN4A.1
- net N$18: now also CX1.1, IC3.OSC2, X2A.2; no longer LED3.BLUE_A, RN5C.1
- net N$19: now also CX2.1, IC3.OSC1, X2A.1; no longer LED3.GREEN_A, RN5B.1
- net N$20: now also N5110.7; no longer LED3.RED_A, RN5A.1
- net N$4: now also C9.2, RN2C.2, RN2D.2; no longer LED.BLUE_A, RN2C.1
- net N$8: now also FB1.P$1; no longer N1.7
- net N$9: now also C8.P$1, FB1.P$2, IC6.T-; no longer LED.GREEN_A, RN2B.1
- net RESET: now also IC3.RESET; no longer N1.1
- net RXD: no longer SV2.3
- net SCK: now also D1.C, IC3.SCK
- net SCL: now also IC1.PC5(ADC5/SCL), U3.SCL; no longer LUXNIR.SCL, LUXRGB.SCL, R15.1, RIR2.1, SV2.6, U1.SCL/VZ
- net SDA: now also IC1.PC4(ADC4/SDA), U3.SDA; no longer LUXNIR.SDA, LUXRGB.SDA, R14.1, RIR1.1, SV2.5, U1.PWM/SDA
- net TXD: no longer SV2.4
- net VCC: now also L2.2, R11.1, R3.1, RL.P$2; no longer J2.1, N1.6, Q5.D, Q6.D, Q7.D, RIR1.2, RIR2.2, SV2.2, THM1.2, U1.VDD
Other:
- note added: "DHT22 - Temp and Humidity"
- note added: "Ethernet"
- note added: "Pressure"
- note added: "Thermistor"
- note removed: "RGB+Clear"
- note removed: "Thermistor: screw terminal"
- note removed: "White + NIR"
- moved on the sheet: C14, RN2A, RN2B, RN2C
