File: sqrwear2.0.sch (EAGLE design)
At the start: 49 parts, among them IC1 ATMEGA328P, IC2 MCP73831, IC4 MCP1700-33, J1 AYZ0202, Q4 BSS123, Q5 BSS123, Q6 BSS123, Q7 BSS123, U1 MLX90614_, X1 USBSMD

Commit message: update
Parts:
- removed C14, C15: 0.1uF, adafruit:C-USC0805
- removed J2: (no value), jumper:JP1E
- removed LED1, LED2, LED3: RGBLED5050, adafruit:RGBLED5050
- removed LUXNIR: TSL2561, microbuilder:TSL2561
- removed LUXRGB: TCS34725, dwbLibrary:TCS34725
- removed N1, SV2: (no value), con-lstb:MA08-1
- removed Q5, Q6, Q7: BSS123, transistor-small-signal:BSS123
- removed R14, R15: 10K, adafruit:R-US_R0805
- removed RIR1, RIR2: 10K, rcl:R-EU_R0805
- removed RN2, RN3, RN4, RN5: (no value), resistor-dil:4R-NEXB38V
- removed RTHM1: 3k, rcl:R-US_R0805
- removed THM1: 1X2-3.5MM, adafruit:1X2-3.5MM
- removed U1: MLX90614_, SparkFun:MLX90614_
- added PAD_10, PAD_3, PAD_A4, PAD_A5, PAD_GND, PAD_VCC: SEWTAP6, LilyPad-Wearables:SEWTAP611
- added PAD_11, PAD_13, PAD_5, PAD_6, PAD_A2, PAD_A3, PAD_TXD: SEWTAP6, LilyPad-Wearables:SEWTAP61
- added PAD_RXD: (no value), LilyPad-Wearables:SEWTAP61
- added Q1, Q2, Q3: BSS123, transistor-small-signal:BSS123
- added R2: 10K, rcl:R-EU_R0805
- added RL: PHOTOCELL, SparkFunNew:PHOTOCELLPTH
- added TEMP: MCP9700, linear:LM50
Connections:
- removed net +3V3: C14.1, C15.1, LUXNIR.3.3V, LUXRGB.VDD, R14.2, R15.2
- removed net BLUE: Q6.S, RN2B.2, RN3B.2, RN4B.2, RN5B.2
- removed net GREEN: Q7.S, RN2C.2, RN3C.2, RN4C.2, RN5C.2
- removed net N$11: LED.RED_A, RN2A.1
- removed net N$12: LED1.BLUE_A, RN3C.1
- removed net N$13: LED1.GREEN_A, RN3B.1
- removed net N$14: LED1.RED_A, RN3A.1
- removed net N$15: LED2.BLUE_A, RN4C.1
- removed net N$16: LED2.GREEN_A, RN4B.1
- removed net N$17: LED2.RED_A, RN4A.1
- removed net N$18: LED3.BLUE_A, RN5C.1
- removed net N$19: LED3.GREEN_A, RN5B.1
- removed net N$20: LED3.RED_A, RN5A.1
- removed net RED: Q5.S, RN2A.2, RN3A.2, RN4A.2, RN5A.2
- removed net RGB-INT: LUXRGB.INT
- removed net SCL: LUXNIR.SCL, LUXRGB.SCL, R15.1, RIR2.1, SV2.6, U1.SCL/VZ
- removed net SDA: LUXNIR.SDA, LUXRGB.SDA, R14.1, RIR1.1, SV2.5, U1.PWM/SDA
- removed net VIS-NIR-ADDR: LUXNIR.ADDRSEL
- removed net VIS-NIR-INT: LUXNIR.INT
- new net SP1: PAD_3.1, Q1.D
- new net SP2: PAD_5.1, Q2.D
- new net SP3: PAD_6.1, Q3.D
- net A0: now also R2.1, RL.P$1; no longer SV2.7
- net A1: now also TEMP.VO; no longer SV2.8
- net A2: now also PAD_A2.1; no longer RTHM1.2, THM1.1
- net A3: now also PAD_A3.1; no longer BTN.S, BTN.S1
- net A4: now also PAD_A4.1
- net A5: now also PAD_A5.1
- net D10: now also PAD_10.1; no longer Q7.G
- net D3: now also Q1.G; no longer N1.3
- net D4: now also BTN.S, BTN.S1; no longer N1.4
- net D5: now also Q2.G; no longer N1.5
- net D6: now also Q3.G; no longer Q5.G
- net D8: now also RN1C.1; no longer Q6.G
- net GND: now also PAD_GND.1, Q1.S, Q2.S, Q3.S, R2.2, TEMP.GND; no longer C14.2, C15.2, LED1.BLUE_C, LED1.GREEN_C, LED1.RED_C, LED2.BLUE_C, LED2.GREEN_C, LED2.RED_C, LED3.BLUE_C, LED3.GREEN_C, LED3.RED_C, LUXNIR.GND, LUXRGB.GND, N1.2, N1.8, RTHM1.1, SV2.1, U1.VSS
- net MISO: now also RN1B.1
- net MOSI: now also PAD_11.1
- net N$4: now also RN1A.2; no longer RN2C.1
- net N$8: now also LED.GREEN_A, RN1B.2; no longer J2.2, N1.7
- net N$9: now also LED.RED_A, RN1C.2; no longer LED.GREEN_A, RN2B.1
- net RESET: no longer N1.1
- net RXD: now also PAD_RXD.1; no longer SV2.3
- net SCK: now also PAD_13.1, RN1A.1
- net TXD: now also PAD_TXD.1; no longer SV2.4
- net VCC: now also PAD_VCC.1, RL.P$2, TEMP.+VS; no longer J2.1, N1.6, Q5.D, Q6.D, Q7.D, RIR1.2, RIR2.2, SV2.2, THM1.2, U1.VDD
Other:
- note removed: "CE"
- note removed: "CLK"
- note removed: "DC"
- note removed: "DIN"
- note removed: "GND"
- note removed: "LIGHT"
- note removed: "RGB+Clear"
- note removed: "RST"
- note removed: "Thermistor: screw terminal"
- note removed: "VCC"
- note removed: "White + NIR"
- moved on the sheet: BTN, LED, Q4, U$1
